Commit message: group 4 vacuum gripper calibration

File: src/abb_irb120_description/urdf/irb120_3_60.xacro (robot description, xacro)
@@ -12,7 +12,13 @@
   <link name="vacuum_tcp_calibrated"/>
   <joint name="tool0-vacuum_tcp_calibrated" type="fixed">
-        <parent link="tool0"/>
-        <child link="vacuum_tcp_calibrated"/>
-        <origin xyz="0 0 0.184" rpy="0 0 ${radians(90)}"/>
-    </joint>
+    <parent link="tool0"/>
+    <child link="vacuum_tcp_calibrated"/>
+    <origin xyz="0 0 0.184" rpy="0 0 ${radians(90)}"/>
+  </joint>
+  <link name="vacuum_tcp_group4"/>
+  <joint name="tool0-vacuum_tcp_group4" type="fixed">
+    <parent link="tool0"/>
+    <child link="vacuum_tcp_group4"/>
+    <origin xyz="0.00201931 -0.000575124 0.179921" rpy="0 0 ${radians(90)}"/>
+  </joint>
 </robot>
